File: ControlUnit/ButtonLEDsController/ButtonLEDsController.kicad_pcb (KiCad board)
At the start: 2 copper layers, 0 parts

Commit message: transistors in schematic taken from 3rd party lib were bad idea because default kicad footprints wouldn't match the pin references in the schematic (were E,B,C - needed to be 1,2,3 instead)
Parts:
- added D1: LED, LEDs:LED_D5.0mm, B.Cu at (21.3, 93.3)
- added D10: LED, LEDs:LED_D5.0mm, B.Cu at (82.2, 93.2)
- added D11: LED, LEDs:LED_D5.0mm, B.Cu at (88.9, 93.2)
- added D12: LED, LEDs:LED_D5.0mm, B.Cu at (96.1, 93.2)
- added D13: DisplayBacklight, LEDs:LED_D5.0mm, F.Cu at (23.2, 76.8)
- added D14: , LEDs:LED_D5.0mm-4, F.Cu at (82.3, 24.9)
- added D15: , LEDs:LED_D5.0mm-4, F.Cu at (82.3, 55.2)
- added D2: LED, LEDs:LED_D5.0mm, B.Cu at (28.1, 93.2)
- added D3: LED, LEDs:LED_D5.0mm, B.Cu at (34.7, 93.2)
- added D4: LED, LEDs:LED_D5.0mm, B.Cu at (41.6, 93.2)
- added D5: LED, LEDs:LED_D5.0mm, B.Cu at (48.4, 93.3)
- added D6: LED, LEDs:LED_D5.0mm, B.Cu at (55.1, 93.3)
- added D7: LED, LEDs:LED_D5.0mm, B.Cu at (62.0, 93.2)
- added D8: LED, LEDs:LED_D5.0mm, B.Cu at (68.8, 93.2)
- added D9: LED, LEDs:LED_D5.0mm, B.Cu at (75.6, 93.2)
- added J1: , Pin_Headers:Pin_Header_Straight_2x15_Pitch2.54mm, F.Cu at (29.1, 25.5)
- added J2: , Pin_Headers:Pin_Header_Straight_1x03_Pitch2.54mm, F.Cu at (18.3, 76.8)
- added J3: , Pin_Headers:Pin_Header_Straight_1x01_Pitch2.54mm, F.Cu at (35.7, 100.8)
- added J4: , Pin_Headers:Pin_Header_Straight_1x01_Pitch2.54mm, F.Cu at (65.5, 16.8)
- added J5: , Pin_Headers:Pin_Header_Straight_1x01_Pitch2.54mm, F.Cu at (52.6, 16.8)
- added J6: , Socket_Strips:Socket_Strip_Straight_1x02_Pitch2.54mm, F.Cu at (51.4, 53.4)
- added Q1: , Power_Integrations:TO-220, F.Cu at (65.8, 43.3)
- added Q2: , TO_SOT_Packages_THT:TO-92_Molded_Narrow, F.Cu at (88.3, 44.6)
- added Q3: , TO_SOT_Packages_THT:TO-92_Molded_Narrow, F.Cu at (71.3, 24.5)
- added Q4: , TO_SOT_Packages_THT:TO-92_Molded_Narrow, F.Cu at (71.4, 30.0)
- added Q5: , TO_SOT_Packages_THT:TO-92_Molded_Narrow, F.Cu at (71.4, 35.6)
- added Q6: , TO_SOT_Packages_THT:TO-92_Molded_Narrow, F.Cu at (71.3, 54.8)
- added Q7: , TO_SOT_Packages_THT:TO-92_Molded_Narrow, F.Cu at (71.4, 60.4)
- added Q8: , TO_SOT_Packages_THT:TO-92_Molded_Narrow, F.Cu at (71.3, 65.8)
- added R1: 10k, Resistors_THT:R_Axial_DIN0204_L3.6mm_D1.6mm_P7.62mm_Horizontal, F.Cu at (70.1, 46.9)
- added R2: 10k, Resistors_THT:R_Axial_DIN0204_L3.6mm_D1.6mm_P7.62mm_Horizontal, F.Cu at (82.6, 43.3)
- added R3: 330, Resistors_THT:R_Axial_DIN0204_L3.6mm_D1.6mm_P7.62mm_Horizontal, F.Cu at (25.8, 85.2)
- added R4: 1k, Resistors_THT:R_Axial_DIN0204_L3.6mm_D1.6mm_P7.62mm_Horizontal, F.Cu at (63.6, 23.3)
- added R5: 1k, Resistors_THT:R_Axial_DIN0204_L3.6mm_D1.6mm_P7.62mm_Horizontal, F.Cu at (63.4, 28.8)
- added R6: 1k, Resistors_THT:R_Axial_DIN0204_L3.6mm_D1.6mm_P7.62mm_Horizontal, F.Cu at (63.4, 34.3)
- added R7: 1k, Resistors_THT:R_Axial_DIN0204_L3.6mm_D1.6mm_P7.62mm_Horizontal, F.Cu at (65.2, 53.5)
- added R8: 1k, Resistors_THT:R_Axial_DIN0204_L3.6mm_D1.6mm_P7.62mm_Horizontal, F.Cu at (65.0, 59.1)
- added R9: 1k, Resistors_THT:R_Axial_DIN0204_L3.6mm_D1.6mm_P7.62mm_Horizontal, F.Cu at (65.0, 64.6)
- added U1: NodeMCU1.0(ESP-12E), NodeMCU:NodeMCU1.0(12-E), F.Cu at (31.1, 45.9)
Routing:
- net +5V: track 0.00 -> 173.6 mm
- net +12V: track 0.00 -> 156.9 mm, vias 0 -> 1
- net MOSFET_DRAIN: track 0.00 -> 135.8 mm
- net Net-(Q2-Pad3): track 0.00 -> 110.9 mm
- net +3V3: track 0.00 -> 72.9 mm, vias 0 -> 1
- net D5: track 0.00 -> 42.2 mm
- net D4: track 0.00 -> 41.9 mm
- net D3: track 0.00 -> 39.0 mm
- net D6: track 0.00 -> 38.9 mm
- net D2: track 0.00 -> 25.8 mm
- net D0: track 0.00 -> 25.3 mm
- net D1: track 0.00 -> 24.5 mm
- net A0: track 0.00 -> 24.0 mm
- net TX: track 0.00 -> 19.7 mm
- net RX: track 0.00 -> 19.7 mm
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- added copper zone on B.Cu, net GND
- added copper zone on F.Cu, net GND
Other:
- board outline added: 100.1 x 90.1 mm
