File: ControlUnit/ButtonLEDsController/ButtonLEDsController.kicad_pcb (KiCad board)
At the start: 2 copper layers, 100.1 x 90.1 mm, 39 parts, among them U1 NodeMCU1.0(ESP-12E)

Commit message: clarify power connector voltages add license information and revisions to boards
Other:
- board text added: "+"
- board text added: "12V"
- board text added: "3.3 V"
- board text added: "5V"
- board text added: "Board layout by CodingSpiderFox License: CERN OHL v1.2"
- board text added: "Rev 0.1"
Changed lines of the file:
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@@
     (links 100)
     (no_connects 3)
-    (area 14.580399 13.615199 114.731001 103.766001)
+    (area 12.4968 13.1572 117.144801 106.273601)
     (thickness 1.6)
-    (drawings 4)
+    (drawings 10)
     (tracks 177)
     (zones 0)
@@
     )
   )
+  (gr_text "Rev 0.1" (at 108.6104 101.5238) (layer Eco2.User)
+    (effects (font (size 1.5 1.5) (thickness 0.3)))
+  )
+  (gr_text "Board layout by CodingSpiderFox\nLicense: CERN OHL v1.2" (at 109.9312 34.2392 90) (layer Eco2.User)
+    (effects (font (size 1.5 1.5) (thickness 0.3)))
+  )
+  (gr_text 12V (at 42.1894 99.9236) (layer Eco2.User)
+    (effects (font (size 1.5 1.5) (thickness 0.3)))
+  )
+  (gr_text + (at 27.3558 75.0062) (layer Eco2.User)
+    (effects (font (size 1.5 1.5) (thickness 0.3)))
+  )
+  (gr_text "3.3 V" (at 49.8348 19.9644) (layer Eco2.User)
+    (effects (font (size 1.5 1.5) (thickness 0.3)))
+  )
+  (gr_text "5V\n" (at 69.1134 18.9484) (layer Eco2.User)
+    (effects (font (size 1.5 1.5) (thickness 0.3)))
+  )
   (gr_line (start 114.681 13.716) (end 114.681 103.716) (angle 90) (layer Edge.Cuts) (width 0.1))
