File: LightingUnit/LightingUnit.kicad_pcb (KiCad board)
At the start: 2 copper layers, 100 x 60 mm, 10 parts, among them U2 IRLZ34

Commit message: clean up, add license info
Parts:
- R3: value Photores -> LDR
Routing:
- net A0: track 91.7 -> 101.9 mm
Other:
- outline, holes or cut-outs redrawn
- board text added: "Board design by CodingSpiderFox License: CERN OHL v1.2"
- board text added: "Rev 0.1"
Changed lines of the file:
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@@
   (general
     (links 49)
-    (no_connects 1)
-    (area 12.624999 13.894999 112.775001 74.045001)
+    (no_connects 0)
+    (area 13.97 12.7 116.840001 74.930001)
     (thickness 1.6)
-    (drawings 5)
-    (tracks 80)
+    (drawings 7)
+    (tracks 81)
     (zones 0)
     (modules 10)
@@
     (pad_to_mask_clearance 0.2)
     (aux_axis_origin 0 0)
-    (grid_origin 27.94 15.24)
     (visible_elements FFFFFF7F)
     (pcbplotparams
@@
     (descr "Through hole pin header")
     (tags "pin header")
-    (fp_text reference P1 (at 2.54 -2.54 180) (layer F.SilkS)
+    (fp_text reference P1 (at 2.54 -2.04 180) (layer F.SilkS)
       (effects (font (size 1 1) (thickness 0.15)))
     )
@@
     (descr "Through hole pin header")
     (tags "pin header")
-    (fp_text reference P2 (at 2.54 -2.54 180) (layer F.SilkS)
+    (fp_text reference P2 (at 0 7.62 180) (layer F.SilkS)
       (effects (font (size 1 1) (thickness 0.15)))
     )
@@
     (descr "Through hole pin header")
     (tags "pin header")
-    (fp_text reference P3 (at 2.54 -2.54 180) (layer F.SilkS)
+    (fp_text reference P3 (at 0 5.08 180) (layer F.SilkS)
       (effects (font (size 1 1) (thickness 0.15)))
     )
@@
     (descr "Through hole pin header")
     (tags "pin header")
-    (fp_text reference P4 (at 2.54 -2.54 180) (layer F.SilkS)
+    (fp_text reference P4 (at 0 5.08 180) (layer F.SilkS)
       (effects (font (size 1 1) (thickness 0.15)))
     )
@@
       (effects (font (size 1 1) (thickness 0.15)))
     )
-    (fp_text value 10k (at 5.08 3.81 270) (layer F.Fab)
+    (fp_text value 10k (at 5.08 2.54 270) (layer F.Fab)
       (effects (font (size 1 1) (thickness 0.15)))
     )
@@
     (descr "Resistance verticale")
     (tags R)
-    (fp_text reference R3 (at -1.016 2.54 180) (layer F.SilkS)
-      (effects (font (size 1 1) (thickness 0.15)))
-    )
-    (fp_text value Photores (at -6.35 0 180) (layer F.Fab)
+    (fp_text reference R3 (at -3.81 2.54 180) (layer F.SilkS)
+      (effects (font (size 1 1) (thickness 0.15)))
+    )
+    (fp_text value LDR (at -5.08 0 180) (layer F.Fab)
       (effects (font (size 1 1) (thickness 0.15)))
     )
@@
       (net 8 D0))
   )
-  (gr_line (start 111.76 13.97) (end 111.76 73.97) (angle 90) (layer Edge.Cuts) (width 0.15))
+  (gr_text "Rev 0.1\n" (at 22.86 71.12) (layer Eco2.User)
+    (effects (font (size 1.5 1.5) (thickness 0.3)))
+  )
+  (gr_text "Board design by CodingSpiderFox\nLicense: CERN OHL v1.2" (at 71.12 16.51) (layer Eco2.User)
+    (effects (font (size 1 1) (thickness 0.1)))
+  )
+  (gr_line (start 85.09 13.97) (end 85.09 73.97) (angle 90) (layer Edge.Cuts) (width 0.15))
   (gr_line (start 15.24 73.66) (end 115.24 73.66) (angle 90) (layer Edge.Cuts) (width 0.15))
   (gr_line (start 52.07 13.97) (end 50.8 13.97) (angle 90) (layer Edge.Cuts) (width 0.15))
@@
   (segment (start 31.75 29.21) (end 46.99 29.21) (width 0.25) (layer F.Cu) (net 5))
   (segment (start 72.39 69.85) (end 80.01 69.85) (width 0.25) (layer F.Cu) (net 6))
+  (segment (start 19.05 24.13) (end 29.21 24.13) (width 0.25) (layer F.Cu) (net 7) (status C00000))
   (segment (start 77.47 45.72) (end 77.47 59.69) (width 0.25) (layer F.Cu) (net 7))
   (segment (start 29.21 24.13) (end 29.21 20.32) (width 0.25) (layer F.Cu) (net 7))

Commit message: add voltage labels
Other:
- board text added: "12V"
- board text added: "3.3V"
- board text added: "5V"
Changed lines of the file:
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@@
     (area 13.97 12.7 116.840001 74.930001)
     (thickness 1.6)
-    (drawings 7)
+    (drawings 10)
     (tracks 81)
     (zones 0)
@@
       (net 8 D0))
   )
+  (gr_text 12V (at 82.55 69.85 90) (layer Eco2.User)
+    (effects (font (size 1 1) (thickness 0.1)))
+  )
+  (gr_text "3.3V\n" (at 67.31 71.12) (layer Eco2.User)
+    (effects (font (size 1 1) (thickness 0.1)))
+  )
+  (gr_text "5V\n\n" (at 57.15 72.39) (layer Eco2.User)
+    (effects (font (size 1 1) (thickness 0.1)))
+  )
   (gr_text "Rev 0.1\n" (at 22.86 71.12) (layer Eco2.User)
